Commit message: fix lio-sam

File: LIO-SAM/config/robot.urdf.xacro (robot description, xacro)
@@ -15,10 +15,10 @@
     <child link="base_link"/>
   </joint>
-  <link name="imu_link"> </link>
+  <!-- <link name="imu_link"> </link>
   <joint name="imu_joint" type="fixed">
     <parent link="base_link" />
     <child link="imu_link" />
     <origin xyz="0 0 0" rpy="0 0 0" />
-  </joint>
+  </joint> -->
   <link name="navsat_link"> </link>
   <joint name="navsat_joint" type="fixed">

File: livox_laser_simulation_RO2/urdf/mid360.xacro (robot description, xacro)
@@ -7,5 +7,5 @@
   <xacro:property name="resolution" value="0.002"/>
   <xacro:property name="noise_mean" value="0.0"/>
-  <xacro:property name="noise_stddev" value="0.01"/>
+  <xacro:property name="noise_stddev" value="0.0"/>
   <xacro:property name="mass" value="0.4" />
   <xacro:property name="length" value="0.1" />
@@ -37,5 +37,5 @@
         <pose>0 0 0 0 0 0</pose>
         <visualize>true</visualize>
-        <update_rate>10</update_rate>
+        <update_rate>50</update_rate>
         <!-- This ray plgin is only for visualization. -->
         <plugin name="${name}_plugin" filename="libros2_livox.so">

File: rm_simulation/urdf/simulation_waking_robot.xacro (robot description, xacro)
@@ -217,9 +217,9 @@
     <sensor name="mid360_imu" type="imu">
       <always_on>true</always_on>
-      <update_rate>100</update_rate>
+      <update_rate>500</update_rate>
       <plugin name="imu_plugin" filename="libgazebo_ros_imu_sensor.so">
         <ros>
           <namespace>/</namespace>
-          <remapping>/out:=/livox/imu</remapping>
+          <remapping>~/out:=/livox/imu</remapping>
         </ros>
         <frame_name>imu_link</frame_name>
