Commit message: fix

File: livox_laser_simulation_RO2/urdf/mid360.xacro (robot description, xacro)
@@ -7,5 +7,5 @@
   <xacro:property name="resolution" value="0.002"/>
   <xacro:property name="noise_mean" value="0.0"/>
-  <xacro:property name="noise_stddev" value="0.0"/>
+  <xacro:property name="noise_stddev" value="0.02"/>
   <xacro:property name="mass" value="0.4" />
   <xacro:property name="length" value="0.1" />

File: rm_simulation/urdf/simulation_waking_robot.xacro (robot description, xacro)
@@ -217,5 +217,5 @@
     <sensor name="mid360_imu" type="imu">
       <always_on>true</always_on>
-      <update_rate>500</update_rate>
+      <update_rate>100</update_rate>
       <plugin name="imu_plugin" filename="libgazebo_ros_imu_sensor.so">
         <ros>
